File: KiCad/T815-DKR-86-Schema/T815-DKR-86-Schema.kicad_sch (KiCad schematic)
At the start: 54 parts, among them M1 RC Model Motor, Q1 BS170, Q10 BS170, Q11 BS170, Q2 BS170, Q7 BS170, Q8 BS170, Q9 BS170, U1 Optocoupler_Module, U3 PWM_MOSFET_Module, U4 ESC - regulator, U5 Step Down to 5V

Commit message: get ready for more clever button class
Parts:
- R17, R18, R19, R20, R5, R6, R7, R8: footprint (none) -> Resistor_THT:R_Axial_DIN0204_L3.6mm_D1.6mm_P7.62mm_Horizontal
Changed lines of the file:
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@@
 	)
 	(junction
-		(at 140.97 93.98)
+		(at 64.77 99.06)
 		(diameter 0)
 		(color 0 0 0 0)
 	)
 	(junction
-		(at 113.03 81.28)
+		(at 140.97 93.98)
 		(diameter 0)
 		(color 0 0 0 0)
 	)
 	(junction
-		(at 52.07 179.07)
+		(at 113.03 81.28)
 		(diameter 0)
 		(color 0 0 0 0)
 	)
 	(junction
-		(at 59.69 99.06)
+		(at 52.07 179.07)
 		(diameter 0)
 		(color 0 0 0 0)
@@
 	(wire
 		(pts
-			(xy 82.55 146.05) (xy 80.01 146.05)
+			(xy 88.9 146.05) (xy 86.36 146.05)
 		)
 		(stroke
@@
 	(wire
 		(pts
-			(xy 67.31 157.48) (xy 67.31 156.21)
+			(xy 72.39 157.48) (xy 72.39 156.21)
 		)
 		(stroke
@@
 	(wire
 		(pts
-			(xy 25.4 99.06) (xy 59.69 99.06)
+			(xy 25.4 99.06) (xy 64.77 99.06)
 		)
 		(stroke
@@
 	(wire
 		(pts
-			(xy 127 102.87) (xy 82.55 102.87)
+			(xy 127 102.87) (xy 88.9 102.87)
 		)
 		(stroke
@@
 	(wire
 		(pts
-			(xy 67.31 167.64) (xy 67.31 168.91)
+			(xy 72.39 167.64) (xy 72.39 168.91)
 		)
 		(stroke
@@
 	(wire
 		(pts
-			(xy 72.39 179.07) (xy 52.07 179.07)
+			(xy 78.74 179.07) (xy 52.07 179.07)
 		)
 		(stroke
@@
 	(wire
 		(pts
-			(xy 67.31 156.21) (xy 52.07 156.21)
-		)
-		(stroke
-			(width 0)
-			(type default)
-		)
-	)
-	(wire
-		(pts
-			(xy 59.69 99.06) (xy 124.46 99.06)
+			(xy 72.39 156.21) (xy 52.07 156.21)
 		)
 		(stroke
@@
 	(wire
 		(pts
-			(xy 72.39 135.89) (xy 72.39 140.97)
+			(xy 78.74 135.89) (xy 78.74 140.97)
 		)
 		(stroke
@@
 	(wire
 		(pts
-			(xy 67.31 168.91) (xy 52.07 168.91)
+			(xy 72.39 168.91) (xy 52.07 168.91)
 		)
 		(stroke
@@
 	(wire
 		(pts
-			(xy 82.55 102.87) (xy 82.55 146.05)
+			(xy 88.9 102.87) (xy 88.9 146.05)
 		)
 		(stroke
@@
 	(wire
 		(pts
-			(xy 59.69 99.06) (xy 59.69 162.56)
+			(xy 64.77 99.06) (xy 64.77 162.56)
 		)
 		(stroke
@@
 	(wire
 		(pts
+			(xy 64.77 99.06) (xy 124.46 99.06)
+		)
+		(stroke
+			(width 0)
+			(type default)
+		)
+	)
+	(wire
+		(pts
 			(xy 93.98 86.36) (xy 102.87 86.36)
 		)
@@
 	(wire
 		(pts
-			(xy 72.39 151.13) (xy 72.39 179.07)
+			(xy 78.74 151.13) (xy 78.74 179.07)
 		)
 		(stroke
@@
 			)
 		)
-		(property "Footprint" ""
+		(property "Footprint" "Resistor_THT:R_Axial_DIN0204_L3.6mm_D1.6mm_P7.62mm_Horizontal"
 			(at 219.202 101.6 90)
 			(effects
@@
 	(symbol
 		(lib_id "Transistor_FET:IRLZ44N")
-		(at 74.93 146.05 180)
+		(at 81.28 146.05 180)
 		(unit 1)
 		(exclude_from_sim no)
@@
 		(dnp no)
 		(property "Reference" "Q7"
-			(at 82.55 143.764 0)
+			(at 88.9 143.764 0)
 			(effects
 				(font
@@
 		)
 		(property "Value" "BS170"
-			(at 82.55 143.256 0)
+			(at 88.9 143.256 0)
 			(effects
 				(font
@@
 		)
 		(property "Footprint" "Package_TO_SOT_THT:TO-220-3_Vertical"
-			(at 69.85 144.145 0)
+			(at 76.2 144.145 0)
 			(effects
 				(font
@@
 		)
 		(property "Datasheet" "https://www.gme.cz/v/1492728/onsemifairchild-bs170-unipolarni-tranzistor"
-			(at 69.85 142.24 0)
+			(at 76.2 142.24 0)
 			(effects
 				(font
@@
 		)
 		(property "Description" "Unipolární tranzistor, N kanál, THT, 60V, 0,5A, 0,83W, TO92"
-			(at 74.93 146.05 0)
+			(at 81.28 146.05 0)
 			(effects
 				(font
@@
 			)
 		)
-		(property "Footprint" ""
+		(property "Footprint" "Resistor_THT:R_Axial_DIN0204_L3.6mm_D1.6mm_P7.62mm_Horizontal"
 			(at 275.082 101.6 90)
 			(effects
@@
 			)
 		)
-		(property "Footprint" ""
+		(property "Footprint" "Resistor_THT:R_Axial_DIN0204_L3.6mm_D1.6mm_P7.62mm_Horizontal"
 			(at 263.652 101.6 90)
 			(effects
@@
 	(symbol
 		(lib_id "power:GND")
-		(at 72.39 135.89 180)
+		(at 78.74 135.89 180)
 		(unit 1)
 		(exclude_from_sim no)
@@
 		(fields_autoplaced yes)
 		(property "Reference" "#PWR015"
-			(at 72.39 129.54 0)
+			(at 78.74 129.54 0)
 			(effects
 				(font
@@
 		)
 		(property "Value" "GND"
-			(at 74.93 134.6199 0)
+			(at 81.28 134.6199 0)
 			(effects
 				(font
@@
 		)
 		(property "Footprint" ""
-			(at 72.39 135.89 0)
+			(at 78.74 135.89 0)
 			(effects
 				(font
@@
 		)
 		(property "Datasheet" ""
-			(at 72.39 135.89 0)
+			(at 78.74 135.89 0)
 			(effects
 				(font
@@
 		)
 		(property "Description" "Power symbol creates a global label with name \"GND\" , ground"
-			(at 72.39 135.89 0)
+			(at 78.74 135.89 0)
 			(effects
 				(font
@@
 			)
 		)
-		(property "Footprint" ""
+		(property "Footprint" "Resistor_THT:R_Axial_DIN0204_L3.6mm_D1.6mm_P7.62mm_Horizontal"
 			(at 196.342 101.6 90)
 			(effects
@@
 			)
 		)
-		(property "Footprint" ""
+		(property "Footprint" "Resistor_THT:R_Axial_DIN0204_L3.6mm_D1.6mm_P7.62mm_Horizontal"
 			(at 230.632 101.6 90)
 			(effects
@@
 			)
 		)
-		(property "Footprint" ""
+		(property "Footprint" "Resistor_THT:R_Axial_DIN0204_L3.6mm_D1.6mm_P7.62mm_Horizontal"
 			(at 252.222 101.6 90)
 			(effects
@@
 			)
 		)
-		(property "Footprint" ""
+		(property "Footprint" "Resistor_THT:R_Axial_DIN0204_L3.6mm_D1.6mm_P7.62mm_Horizontal"
 			(at 207.772 101.6 90)
 			(effects
@@
 			)
 		)
-		(property "Footprint" ""
+		(property "Footprint" "Resistor_THT:R_Axial_DIN0204_L3.6mm_D1.6mm_P7.62mm_Horizontal"
 			(at 240.792 101.6 90)
 			(effects
@@
 	(symbol
 		(lib_id "Transistor_FET:IRLZ44N")
-		(at 64.77 162.56 0)
+		(at 69.85 162.56 0)
 		(unit 1)
 		(exclude_from_sim no)
@@
 		(dnp no)
 		(property "Reference" "Q1"
-			(at 57.15 164.846 0)
+			(at 62.23 164.846 0)
 			(effects
 				(font
@@
 		)
 		(property "Value" "BS170"
-			(at 57.15 165.354 0)
+			(at 62.23 165.354 0)
 			(effects
 				(font
@@
 		)
 		(property "Footprint" "Package_TO_SOT_THT:TO-220-3_Vertical"
-			(at 69.85 164.465 0)
+			(at 74.93 164.465 0)
 			(effects
 				(font
@@
 		)
 		(property "Datasheet" "https://www.gme.cz/v/1492728/onsemifairchild-bs170-unipolarni-tranzistor"
-			(at 69.85 166.37 0)
+			(at 74.93 166.37 0)
 			(effects
 				(font
@@
 		)
 		(property "Description" "Unipolární tranzistor, N kanál, THT, 60V, 0,5A, 0,83W, TO92"
-			(at 64.77 162.56 0)
+			(at 69.85 162.56 0)
 			(effects
 				(font

Commit message: new version of schema using new schematic layouts to be able make good pcb layout. Typicaly led arrays are realies as connector with common ground, not a many plus and minus wires.
Parts:
- added J1: PWM Steering, Connector_PinHeader_2.54mm:PinHeader_1x03_P2.54mm_Vertical, symbol Connector_Generic:Conn_01x03
- added J2: PWM Throttle, Connector_PinHeader_2.54mm:PinHeader_1x03_P2.54mm_Vertical, symbol Connector_Generic:Conn_01x03
- added J3: PWM 3.ch.button, Connector_PinHeader_2.54mm:PinHeader_1x03_P2.54mm_Vertical, symbol Connector_Generic:Conn_01x03
- Q1, Q10, Q11, Q2, Q7, Q8, Q9: footprint Package_TO_SOT_THT:TO-220-3_Vertical -> Package_TO_SOT_THT:TO-92L_Inline_Wide
- R1, R10, R11, R12, R13, R14, R15, R2, R3, R4: footprint (none) -> Resistor_THT:R_Axial_DIN0204_L3.6mm_D1.6mm_P2.54mm_Vertical
- R17, R18, R19, R20, R5, R6, R7, R8: footprint Resistor_THT:R_Axial_DIN0204_L3.6mm_D1.6mm_P7.62mm_Horizontal -> Resistor_THT:R_Axial_DIN0204_L3.6mm_D1.6mm_P2.54mm_Vertical
- renumbered D4 to DI1, D3 to DI2, D10 to DIB1, D11 to DIB2, D2 to DO1, D1 to DO2, D13 to DOB1, D12 to DOB2, D14 to DPwmState1, D15 to DR1, D16 to DR2, D17 to DR3, D18 to DR4, D8 to DR5, D7 to DR6, D6 to DR7, D5 to DR8
Connections:
- net GND: now also J1.3 (Pin_3), J2.3 (Pin_3), J3.3 (Pin_3)
- net at A1.12 (D9): now also J3.1 (Pin_1)
- net at A1.13 (D10): now also J2.1 (Pin_1)
- net at A1.14 (D11): now also J1.1 (Pin_1)
Other:
- moved on the sheet: DI1, DI2, DO1, DO2, DPwmState1, DR1, DR2, DR3, DR4, DR5, DR6, DR7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
